Commit message: model updated with wheels

File: osmose_description/urdf/base.urdf (robot description, URDF)
Before this commit: robot osmose, 1 links, 0 joints
Links:
- added link left_wheel, mass 5; collision mesh filename=file://$(find osmose_description)/meshes/Wheels.stl scale=1 1 1; visual mesh filename=file://$(find osmose_description)/meshes/Wheels.stl scale=1 1 1
- added link right_wheel, mass 5; collision mesh filename=file://$(find osmose_description)/meshes/Wheels.stl scale=1 1 1; visual mesh filename=file://$(find osmose_description)/meshes/Wheels.stl scale=1 1 1
Joints:
- added joint left_wheel_hinge: type continuous, parent base_link, child left_wheel, origin xyz=0.053 0.1225 -0.13 rpy=0 0 0, axis 0 1 0, limit effort=10000 velocity=1000
- added joint right_wheel_hinge: type continuous, parent base_link, child right_wheel, origin xyz=0.053 -0.1225 -0.13 rpy=0 0 0, axis 0 1 0, limit effort=10000 velocity=1000

Commit message: gazebo_wheels link imp

File: osmose_description/urdf/base.urdf (robot description, URDF)
Before this commit: robot osmose, 3 links, 2 joints
Joints:
- joint left_wheel_hinge: origin xyz=0.053 0.1225 -0.13 rpy=0 0 0 -> xyz=0.053 -0.1225 -0.13 rpy=0 0 0
- joint right_wheel_hinge: origin xyz=0.053 -0.1225 -0.13 rpy=0 0 0 -> xyz=0.053 0.1225 -0.13 rpy=0 0 0

Commit message: cmd as m/s ifor each wheels instead of twist to both
http://wiki.ros.org/differential_drive

with virtual joystick, adapted to python3 and noetic

File: osmose_description/urdf/base.urdf (robot description, URDF)
Before this commit: robot osmose, 3 links, 2 joints
Links:
- removed link left_wheel
- removed link right_wheel
- added link lwheel, mass 5; collision mesh filename=file://$(find osmose_description)/meshes/Wheels.stl scale=1 1 1; visual mesh filename=file://$(find osmose_description)/meshes/Wheels.stl scale=1 1 1
- added link rwheel, mass 5; collision mesh filename=file://$(find osmose_description)/meshes/Wheels.stl scale=1 1 1; visual mesh filename=file://$(find osmose_description)/meshes/Wheels.stl scale=1 1 1
Joints:
- joint left_wheel_hinge: child left_wheel -> lwheel
- joint right_wheel_hinge: child right_wheel -> rwheel
